File: STM32F103.kicad_sch (KiCad schematic)
At the start: 15 parts, among them SW4 SW_SPST, U2 STM32F103CBTx, Y1 12MHz

Commit message: 3/30
Parts:
- renumbered C5 to C10, C6 to C11, C7 to C2, C8 to C3, C9 to C4, C10 to C5, C13 to C6, C15 to C7, C18 to C8, C4 to C9, R12 to R5, SW4 to SW1
Connections:
- net INDICATOR_RED: now reaches U2.21 (PB10)
- net INDICATOR_YELLOW: now reaches U2.22 (PB11)
- net INDICATOR_GREEN: now reaches U2.25 (PB12)
- net INDICATOR_BUZZER: now reaches U2.26 (PB13)
- no-connect marks 27 -> 24

Commit message: 4/2
Parts:
- removed L1: 27n, Inductor_SMD:L_0603_1608Metric, symbol Device:L
- added FB1: FerriteBead, Inductor_SMD:L_0603_1608Metric, symbol Device:FerriteBead_Small
- C8: value 100n -> 0.1u
- SW1: value SW_SPST -> SPST_SW; footprint Button_Switch_THT:SW_PUSH_6mm_H7.3mm -> Button_Switch_SMD:SW_Push_1P1T_XKB_TS-1187A
- renumbered R5 to R9
Connections:
- net CAN_RX: now also U2.45 (PB8); no longer U2.32 (PA11)
- net CAN_TX: now also U2.46 (PB9); no longer U2.33 (PA12)
- net VDD: now also FB1.1
- net VDDA: now also FB1.2
- new net USB_D+: U2.33 (PA12)
- new net USB_D-: U2.32 (PA11)
- no-connect marks 24 -> 22

Commit message: 4/13 product update
Parts:
- FB1: LCSC (none) -> C1002
- SW1: LCSC (none) -> C318884
- U2: LCSC (none) -> C8734
- Y1: LCSC (none) -> C9002
Changed lines of the file:
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@@
+      (effects (font (size 1.27 1.27)) hide)
+    )
+    (property "LCSC" "C318884" (at 29.21 86.36 0)
       (effects (font (size 1.27 1.27)) hide)
     )
@@
     )
     (property "Datasheet" "https://www.st.com/resource/en/datasheet/stm32f103cb.pdf" (at 110.49 110.49 0)
+      (effects (font (size 1.27 1.27)) hide)
+    )
+    (property "LCSC" "C8734" (at 110.49 110.49 0)
       (effects (font (size 1.27 1.27)) hide)
     )
@@
       (effects (font (size 1.27 1.27)) hide)
     )
+    (property "LCSC" "C1002" (at 160.02 72.39 0)
+      (effects (font (size 1.27 1.27)) hide)
+    )
     (pin "1")
     (pin "2")
@@
       (effects (font (size 1.27 1.27)) hide)
     )
+    (property "LCSC" "C9002" (at 62.23 99.06 0)
+      (effects (font (size 1.27 1.27)) hide)
+    )
