File: EMS.kicad_sch (KiCad schematic)
At the start: 19 parts, among them J2 Conn_01x02, J3 Conn_01x02, J4 Conn_01x02, J5 Conn_01x04, Q1 Q_NMOS_GDS, Q2 Q_PMOS_GSD, Q3 Q_NMOS_GSD

Commit message: 3/30
Parts:
- added D5: D_Zener, symbol Device:D_Zener
- R10: renamed from R2; value R -> 100
- R12: renamed from R3; value R -> 10k
- R9: renamed from R1; value R -> 10k
- renumbered D1 to D4, D2 to D6, J3 to J10, J4 to J11, J5 to J12, J2 to J9, Q1 to Q2, Q2 to Q3, Q3 to Q4, R4 to R11, R5 to R13, R8 to R14, R6 to R15, R7 to R16
Connections:
- net +12V: now also D4.1 (K); no longer D4.2 (A)
- net at D6.1 (K), J9.2 (Pin_2), Q2.2 (D): now also D5.1 (K); no longer D4.1 (K)
- new net: D4.2 (A), D5.2 (A)
Other:
- moved on the sheet: D4, D6, J10, R9

Commit message: 4/2
Parts:
- removed J12: Conn_01x04, symbol Connector_Generic:Conn_01x04
- added J14, J15: Remote_SW, TerminalBlock:TerminalBlock_bornier-2_P5.08mm, symbol Connector_Generic:Conn_01x02
- D5: renamed from D4; footprint (none) -> Diode_SMD:D_SMA
- D6: renamed from D5; footprint (none) -> Diode_SMD:D_SOD-123
- D7: renamed from D6; footprint (none) -> LED_SMD:LED_0603_1608Metric
- J11: renamed from J9; value Conn_01x02 -> Relay; footprint (none) -> Connector_JST:JST_XA_B02B-XASK-1_1x02_P2.50mm_Vertical
- J12: renamed from J10; value Conn_01x02 -> EMS_SW; footprint (none) -> Connector_JST:JST_XA_B02B-XASK-1_1x02_P2.50mm_Vertical
- J13: renamed from J11; value Conn_01x02 -> EMS_SW; footprint (none) -> Connector_JST:JST_XA_B02B-XASK-1_1x02_P2.50mm_Vertical
- JP1, JP2: value Jumper_2_Open -> EMS_Jumper; footprint (none) -> Connector_PinHeader_2.54mm:PinHeader_1x02_P2.54mm_Vertical
- Q2, Q3: footprint (none) -> Package_TO_SOT_SMD:SOT-23
- R13: renamed from R9; footprint (none) -> Resistor_SMD:R_0603_1608Metric
- R14: renamed from R10; footprint (none) -> Resistor_SMD:R_0603_1608Metric
- R15: renamed from R11; value R -> 10k; footprint (none) -> Resistor_SMD:R_0603_1608Metric
- R16: renamed from R12; footprint (none) -> Resistor_SMD:R_0603_1608Metric
- R17: renamed from R13; value R -> 2k; footprint (none) -> Resistor_SMD:R_0603_1608Metric
- R18: renamed from R14; footprint Resistor_SMD:R_0603_1608Metric_Pad0.98x0.95mm_HandSolder -> Resistor_SMD:R_0603_1608Metric
- R19: renamed from R15; footprint Resistor_SMD:R_0603_1608Metric_Pad0.98x0.95mm_HandSolder -> Resistor_SMD:R_0603_1608Metric
- R20: renamed from R16; footprint Resistor_SMD:R_0603_1608Metric_Pad0.98x0.95mm_HandSolder -> Resistor_SMD:R_0603_1608Metric
Connections:
- net +12V: now also J15.2 (Pin_2)
- net GND: now also J14.1 (Pin_1)
- net at R17.1: now also J15.1 (Pin_1)
Other:
- moved on the sheet: R16

Commit message: 4/12
Parts:
- added JP3: EMS_Jumper, Connector_PinHeader_2.54mm:PinHeader_1x02_P2.54mm_Vertical, symbol Jumper:Jumper_2_Open
Connections:
- net GND: now also JP3.2 (B)
- net at J15.1 (Pin_1), R17.1: now also JP3.1 (A)
Changed lines of the file:
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@@
   (junction (at 168.91 68.58) (diameter 0) (color 0 0 0 0)
   )
+  (junction (at 86.36 104.14) (diameter 0) (color 0 0 0 0)
+  )
   (junction (at 124.46 73.66) (diameter 0) (color 0 0 0 0)
   )
   (junction (at 147.32 140.97) (diameter 0) (color 0 0 0 0)
+  )
+  (junction (at 92.71 100.33) (diameter 0) (color 0 0 0 0)
   )
   (no_connect (at 88.9 96.52))
@@
     (stroke (width 0) (type default))
   )
+  (wire (pts (xy 119.38 85.09) (xy 119.38 104.14))
+    (stroke (width 0) (type default))
+  )
   (wire (pts (xy 168.91 78.74) (xy 168.91 87.63))
     (stroke (width 0) (type default))
@@
     (stroke (width 0) (type default))
   )
+  (wire (pts (xy 109.22 100.33) (xy 109.22 85.09))
+    (stroke (width 0) (type default))
+  )
   (wire (pts (xy 168.91 41.91) (xy 168.91 45.72))
     (stroke (width 0) (type default))
@@
     (stroke (width 0) (type default))
   )
+  (wire (pts (xy 92.71 100.33) (xy 109.22 100.33))
+    (stroke (width 0) (type default))
+  )
   (wire (pts (xy 64.77 73.66) (xy 64.77 77.47))
     (stroke (width 0) (type default))
@@
   )
   (wire (pts (xy 124.46 73.66) (xy 133.35 73.66))
+    (stroke (width 0) (type default))
+  )
+  (wire (pts (xy 119.38 104.14) (xy 86.36 104.14))
     (stroke (width 0) (type default))
   )
@@
         )
       )
+    )
+  )
+  (symbol (lib_id "Jumper:Jumper_2_Open") (at 114.3 85.09 0) (unit 1)
+    (in_bom yes) (on_board yes) (dnp no) (fields_autoplaced)
+    (property "Reference" "JP3" (at 114.3 78.74 0)
+      (effects (font (size 1.27 1.27)))
+    )
+    (property "Value" "EMS_Jumper" (at 114.3 81.28 0)
+      (effects (font (size 1.27 1.27)))
+    )
+    (property "Footprint" "Connector_PinHeader_2.54mm:PinHeader_1x02_P2.54mm_Vertical" (at 114.3 85.09 0)
+      (effects (font (size 1.27 1.27)) hide)
+    )
+    (property "Datasheet" "~" (at 114.3 85.09 0)
+      (effects (font (size 1.27 1.27)) hide)
+    )
+    (pin "1")
+    (pin "2")
+    (instances
+      (project "tsukuba_challenge"
+        (path "/55f88ae9-9831-47be-a185-734020e38c84/38ab94c1-3455-4061-8471-40bae2451452"
+          (reference "JP3") (unit 1)
+        )
+      )

Commit message: 4/13 product update
Parts:
- D5: footprint Diode_SMD:D_SMA -> my_pretty:SOD-123FL; JLCPCB Rotation Offset (none) -> 180; LCSC (none) -> C64898
- D6: LCSC (none) -> C19077414
- D7: LCSC (none) -> C2286
- J11, J12, J13, J14, J15, JP1, JP2, JP3: now left out of the parts list
- Q2, Q4: LCSC (none) -> C7420347
- Q3: LCSC (none) -> C15127
Changed lines of the file:
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@@
       (effects (font (size 1.27 1.27)) (justify left))
     )
-    (property "Footprint" "Diode_SMD:D_SMA" (at 180.34 50.8 0)
+    (property "Footprint" "my_pretty:SOD-123FL" (at 180.34 50.8 0)
       (effects (font (size 1.27 1.27)) hide)
     )
@@
       (effects (font (size 1.27 1.27)) hide)
     )
+    (property "LCSC" "C64898" (at 180.34 50.8 0)
+      (effects (font (size 1.27 1.27)) hide)
+    )
+    (property "JLCPCB Rotation Offset" "180" (at 180.34 50.8 90)
+      (effects (font (size 1.27 1.27)) hide)
+    )
     (pin "1")
     (pin "2")
@@
   )
   (symbol (lib_id "Connector_Generic:Conn_01x02") (at 86.36 91.44 90) (unit 1)
-    (in_bom yes) (on_board yes) (dnp no)
+    (in_bom no) (on_board yes) (dnp no)
     (property "Reference" "J14" (at 80.01 86.36 90)
       (effects (font (size 1.27 1.27)) (justify right))
@@
   )
   (symbol (lib_id "Connector_Generic:Conn_01x02") (at 118.11 63.5 90) (unit 1)
-    (in_bom yes) (on_board yes) (dnp no)
+    (in_bom no) (on_board yes) (dnp no)
     (property "Reference" "J13" (at 125.73 62.23 90)
       (effects (font (size 1.27 1.27)) (justify right))
@@
     )
     (property "Datasheet" "~" (at 166.37 73.66 0)
+      (effects (font (size 1.27 1.27)) hide)
+    )
+    (property "LCSC" "C7420347" (at 166.37 73.66 0)
       (effects (font (size 1.27 1.27)) hide)
     )
@@
   )
   (symbol (lib_id "Connector_Generic:Conn_01x02") (at 97.79 63.5 90) (unit 1)
-    (in_bom yes) (on_board yes) (dnp no)
+    (in_bom no) (on_board yes) (dnp no)
     (property "Reference" "J12" (at 86.36 62.23 90)
       (effects (font (size 1.27 1.27)) (justify right))
@@
   )
   (symbol (lib_id "Connector_Generic:Conn_01x02") (at 187.96 40.64 90) (unit 1)
-    (in_bom yes) (on_board yes) (dnp no) (fields_autoplaced)
+    (in_bom no) (on_board yes) (dnp no) (fields_autoplaced)
     (property "Reference" "J11" (at 193.04 39.37 90)
       (effects (font (size 1.27 1.27)) (justify right))
@@
   )
   (symbol (lib_id "Jumper:Jumper_2_Open") (at 119.38 55.88 0) (unit 1)
-    (in_bom yes) (on_board yes) (dnp no) (fields_autoplaced)
+    (in_bom no) (on_board yes) (dnp no) (fields_autoplaced)
     (property "Reference" "JP2" (at 119.38 49.53 0)
       (effects (font (size 1.27 1.27)))
@@
   )
   (symbol (lib_id "Jumper:Jumper_2_Open") (at 114.3 85.09 0) (unit 1)
-    (in_bom yes) (on_board yes) (dnp no) (fields_autoplaced)
+    (in_bom no) (on_board yes) (dnp no) (fields_autoplaced)
     (property "Reference" "JP3" (at 114.3 78.74 0)
       (effects (font (size 1.27 1.27)))
@@
   )
   (symbol (lib_id "Connector_Generic:Conn_01x02") (at 92.71 91.44 90) (unit 1)
-    (in_bom yes) (on_board yes) (dnp no)
+    (in_bom no) (on_board yes) (dnp no)
     (property "Reference" "J15" (at 91.44 86.36 90)
       (effects (font (size 1.27 1.27)) (justify right))
@@
     )
     (property "Datasheet" "~" (at 168.91 62.23 0)
+      (effects (font (size 1.27 1.27)) hide)
+    )
+    (property "LCSC" "C2286" (at 168.91 62.23 0)
       (effects (font (size 1.27 1.27)) hide)
     )
@@
       (effects (font (size 1.27 1.27)) hide)
     )
+    (property "LCSC" "C7420347" (at 153.67 140.97 0)
+      (effects (font (size 1.27 1.27)) hide)
+    )
     (pin "1")
     (pin "2")
@@
       (effects (font (size 1.27 1.27)) hide)
     )
+    (property "LCSC" "C19077414" (at 185.42 55.88 0)
+      (effects (font (size 1.27 1.27)) hide)
+    )
     (pin "1")
     (pin "2")
@@
   )
   (symbol (lib_id "Jumper:Jumper_2_Open") (at 99.06 55.88 0) (unit 1)
-    (in_bom yes) (on_board yes) (dnp no) (fields_autoplaced)
+    (in_bom no) (on_board yes) (dnp no) (fields_autoplaced)
     (property "Reference" "JP1" (at 99.06 49.53 0)
       (effects (font (size 1.27 1.27)))
@@
       (effects (font (size 1.27 1.27)) hide)
     )
+    (property "LCSC" "C15127" (at 77.47 76.2 0)
+      (effects (font (size 1.27 1.27)) hide)
+    )

Commit message: ✨feat:f302
Parts:
- removed Q2: Q_NMOS_GDS, Package_TO_SOT_SMD:SOT-23, symbol Device:Q_NMOS_GDS
- added Q2: Q_NMOS_GSD, Package_TO_SOT_SMD:SOT-23, symbol Device:Q_NMOS_GSD
Connections:
- net GND: now also Q2.2 (S)
- net at R14.2, R16.2: now also Q2.1 (G)
- net at D6.1 (K), D7.1 (K), J11.2 (Pin_2): now also Q2.3 (D)
Changed lines of the file:
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@@
   (junction (at 93.98 73.66) (diameter 0) (color 0 0 0 0)
   )
+  (junction (at 168.91 68.58) (diameter 0) (color 0 0 0 0)
+  )
   (junction (at 133.35 73.66) (diameter 0) (color 0 0 0 0)
   )
@@
   )
   (junction (at 180.34 45.72) (diameter 0) (color 0 0 0 0)
-  )
-  (junction (at 168.91 68.58) (diameter 0) (color 0 0 0 0)
   )
   (junction (at 86.36 104.14) (diameter 0) (color 0 0 0 0)
@@
     )
   )
-  (symbol (lib_id "Device:Q_NMOS_GDS") (at 166.37 73.66 0) (unit 1)
-    (in_bom yes) (on_board yes) (dnp no) (fields_autoplaced)
-    (property "Reference" "Q2" (at 172.085 72.39 0)
-      (effects (font (size 1.27 1.27)) (justify left))
-    )
-    (property "Value" "Q_NMOS_GDS" (at 172.085 74.93 0)
-      (effects (font (size 1.27 1.27)) (justify left))
-    )
-    (property "Footprint" "Package_TO_SOT_SMD:SOT-23" (at 171.45 71.12 0)
-      (effects (font (size 1.27 1.27)) hide)
-    )
-    (property "Datasheet" "~" (at 166.37 73.66 0)
-      (effects (font (size 1.27 1.27)) hide)
-    )
-    (property "LCSC" "C7420347" (at 166.37 73.66 0)
-      (effects (font (size 1.27 1.27)) hide)
-    )
-    (pin "1")
-    (pin "2")
-    (pin "3")
-    (instances
-      (project "tsukuba_challenge"
-        (path "/55f88ae9-9831-47be-a185-734020e38c84/38ab94c1-3455-4061-8471-40bae2451452"
-          (reference "Q2") (unit 1)
-        )
-      )
-    )
-  )
   (symbol (lib_id "Device:R") (at 147.32 147.32 0) (mirror y) (unit 1)
     (in_bom yes) (on_board yes) (dnp no) (fields_autoplaced)
@@
         )
       )
+      (project "schematic_PWRcutoff"
+        (path "/9e89b938-308a-42c1-b814-ac47b1ea682c/6a93618c-3932-4643-922b-919eb2d9df4b"
+          (reference "Q6") (unit 1)
+        )
+      )
+    )
+  )
+  (symbol (lib_id "Device:Q_NMOS_GSD") (at 166.37 73.66 0) (unit 1)
+    (in_bom yes) (on_board yes) (dnp no)
+    (property "Reference" "Q2" (at 172.72 72.39 0)
+      (effects (font (size 1.27 1.27)) (justify left))
+    )
+    (property "Value" "Q_NMOS_GSD" (at 172.72 74.93 0)
+      (effects (font (size 1.27 1.27)) (justify left))
+    )
+    (property "Footprint" "Package_TO_SOT_SMD:SOT-23" (at 171.45 71.12 0)
+      (effects (font (size 1.27 1.27)) hide)
+    )
+    (property "Datasheet" "~" (at 166.37 73.66 0)
+      (effects (font (size 1.27 1.27)) hide)
+    )
+    (property "LCSC" "C7420347" (at 166.37 73.66 0)
+      (effects (font (size 1.27 1.27)) hide)
+    )
+    (pin "1")
+    (pin "2")
+    (pin "3")
+    (instances
+      (project "tsukuba_challenge"
+        (path "/55f88ae9-9831-47be-a185-734020e38c84/38ab94c1-3455-4061-8471-40bae2451452"
+          (reference "Q2") (unit 1)
+        )
+      )
