File: EMS.kicad_sch (KiCad schematic)
At the start: 22 parts, among them J11 Relay, J12 EMS_SW, J13 EMS_SW, J14 Remote_SW, J15 Remote_SW, Q2 Q_NMOS_GSD, Q3 Q_PMOS_GSD, Q4 Q_NMOS_GSD

Commit message: 6/29
Parts:
- R13, R15, R16, R18, R20: LCSC (none) -> C25804
- R14, R19: LCSC (none) -> C22775
- R17: LCSC (none) -> C22975
Changed lines of the file:
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@@
+      (effects (font (size 1.27 1.27)) hide)
+    )
+    (property "LCSC" "C25804" (at 156.21 125.73 0)
       (effects (font (size 1.27 1.27)) hide)
     )
@@
       (effects (font (size 1.27 1.27)) hide)
     )
+    (property "LCSC" "C22775" (at 152.4 73.66 0)
+      (effects (font (size 1.27 1.27)) hide)
+    )
     (pin "1")
     (pin "2")
@@
       (effects (font (size 1.27 1.27)) hide)
     )
+    (property "LCSC" "C25804" (at 147.32 147.32 0)
+      (effects (font (size 1.27 1.27)) hide)
+    )
     (pin "1")
     (pin "2")
@@
       (effects (font (size 1.27 1.27)) hide)
     )
+    (property "LCSC" "C25804" (at 160.02 81.28 0)
+      (effects (font (size 1.27 1.27)) hide)
+    )
     (pin "1")
     (pin "2")
@@
     )
     (property "Datasheet" "~" (at 77.47 93.98 0)
+      (effects (font (size 1.27 1.27)) hide)
+    )
+    (property "LCSC" "C22975" (at 77.47 93.98 0)
       (effects (font (size 1.27 1.27)) hide)
     )
@@
     )
     (property "Datasheet" "~" (at 168.91 52.07 0)
+      (effects (font (size 1.27 1.27)) hide)
+    )
+    (property "LCSC" "C25804" (at 168.91 52.07 0)
       (effects (font (size 1.27 1.27)) hide)
     )
@@
       (effects (font (size 1.27 1.27)) hide)
     )
+    (property "LCSC" "C22775" (at 140.97 140.97 0)
+      (effects (font (size 1.27 1.27)) hide)
+    )
     (pin "1")
     (pin "2")
@@
       (effects (font (size 1.27 1.27)) hide)
     )
+    (property "LCSC" "C25804" (at 64.77 81.28 0)
+      (effects (font (size 1.27 1.27)) hide)
+    )
