File: power.kicad_sch (KiCad schematic)
At the start: 9 parts, among them U1 XC6206P332MR, U4 L7805

Commit message: 3/30
Parts:
- removed C2: 3.3u, symbol Device:C_Small
- removed C3: 4.7u, symbol Device:C_Polarized
- removed PS1: MIWI06-24S12, my_pretty:MIWI06_S, symbol my_library:MIWI06-24S12
- added C12: 22u, symbol Device:C_Small
- added C13: 120u, symbol Device:C_Polarized
- added D1, D2, D3: LED, symbol Device:LED
- added PS1: CCG30-24-12S_P, my_pretty:CCG304815S, symbol my_library:CCG30-24-12S_P
- added R6: 10k, symbol Device:R
- added R7: 3.3k, symbol Device:R
- added R8: 1.2k, symbol Device:R
- renumbered C1 to C14, C11 to C15, C12 to C16, C14 to C17, U4 to U3, U1 to U4
Connections:
- net +12V: now also C12.1, PS1.4 (+VOUT), R6.1
- net +3.3V: now also R8.1
- net +5V: now also R7.1
- net +BATT: now also C13.1, PS1.3 (+VIN)
- net GND: now also C12.2, D1.1 (K), D2.1 (K), D3.1 (K), PS1.6 (-VOUT)
- net GNDPWR: now also C13.2, PS1.2 (-VIN)
- new net: D2.2 (A), R7.2
- new net: D3.2 (A), R8.2
- new net: D1.2 (A), R6.2
- no-connect marks 0 -> 2

Commit message: 4/2
Parts:
- C12, C14, C15, C16, C17: footprint (none) -> Capacitor_SMD:C_0603_1608Metric
- C13: footprint (none) -> Capacitor_SMD:CP_Elec_6.3x7.7
- D2: renamed from D1; footprint (none) -> LED_SMD:LED_0603_1608Metric
- D3: renamed from D2; footprint (none) -> LED_SMD:LED_0603_1608Metric
- D4: renamed from D3; footprint (none) -> LED_SMD:LED_0603_1608Metric
- R10: renamed from R6; footprint (none) -> Resistor_SMD:R_0603_1608Metric
- R11: renamed from R7; footprint (none) -> Resistor_SMD:R_0603_1608Metric
- R12: renamed from R8; footprint (none) -> Resistor_SMD:R_0603_1608Metric

Commit message: 4/12
Parts:
- C13: value 120u -> 100u; LCSC (none) -> C5355875
Changed lines of the file:
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@@
       (effects (font (size 1.27 1.27)) (justify left))
     )
-    (property "Value" "120u" (at 57.15 57.15 0)
+    (property "Value" "100u" (at 57.15 57.15 0)
       (effects (font (size 1.27 1.27)) (justify left))
     )
@@
       (effects (font (size 1.27 1.27)) hide)
     )
+    (property "LCSC" "C5355875" (at 66.04 57.15 0)
+      (effects (font (size 1.27 1.27)) hide)
+    )

Commit message: 4/13 product update
Parts:
- D2, D3, D4: LCSC (none) -> C2286
- PS1: now left out of the parts list
- U3: JLCPCB Position Offset (none) -> -1.5,0; LCSC (none) -> C58069
- U4: LCSC (none) -> C5446
Changed lines of the file:
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@@
+      (effects (font (size 1.27 1.27)) hide)
+    )
+    (property "LCSC" "C58069" (at 140.97 53.34 0)
+      (effects (font (size 1.27 1.27)) hide)
+    )
+    (property "JLCPCB Position Offset" "-1.5,0" (at 140.97 53.34 0)
       (effects (font (size 1.27 1.27)) hide)
     )
@@
       (effects (font (size 1.27 1.27)) hide)
     )
+    (property "LCSC" "C2286" (at 242.57 55.88 0)
+      (effects (font (size 1.27 1.27)) hide)
+    )
     (pin "1")
     (pin "2")
@@
   )
   (symbol (lib_id "my_library:CCG30-24-12S_P") (at 72.39 48.26 0) (unit 1)
-    (in_bom yes) (on_board yes) (dnp no) (fields_autoplaced)
+    (in_bom no) (on_board yes) (dnp no) (fields_autoplaced)
     (property "Reference" "PS1" (at 87.63 40.64 0)
       (effects (font (size 1.27 1.27)))
@@
       (effects (font (size 1.27 1.27)) hide)
     )
+    (property "LCSC" "C5446" (at 181.61 53.34 0)
+      (effects (font (size 1.27 1.27)) hide)
+    )
     (pin "1")
     (pin "2")
@@
     )
     (property "Datasheet" "~" (at 219.71 55.88 0)
+      (effects (font (size 1.27 1.27)) hide)
+    )
+    (property "LCSC" "C2286" (at 219.71 55.88 0)
       (effects (font (size 1.27 1.27)) hide)
     )
@@
       (effects (font (size 1.27 1.27)) hide)
     )
+    (property "LCSC" "C2286" (at 231.14 55.88 0)
+      (effects (font (size 1.27 1.27)) hide)
+    )

Commit message: product data
Parts:
- C12: footprint Capacitor_SMD:C_0603_1608Metric -> Capacitor_SMD:C_1206_3216Metric; LCSC (none) -> C12891
Changed lines of the file:
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@@
       (effects (font (size 1.27 1.27)) (justify left))
     )
-    (property "Footprint" "Capacitor_SMD:C_0603_1608Metric" (at 110.49 55.88 0)
+    (property "Footprint" "Capacitor_SMD:C_1206_3216Metric" (at 110.49 55.88 0)
       (effects (font (size 1.27 1.27)) hide)
     )
@@
       (effects (font (size 1.27 1.27)) hide)
     )
+    (property "LCSC" "C12891" (at 110.49 55.88 0)
+      (effects (font (size 1.27 1.27)) hide)
+    )

Commit message: ✨feat:f302
Parts:
- PS1: value CCG30-24-12S_P -> CCG30-24-12S
Connections:
- net GNDPWR: now also PS1.1 (RC)
- no-connect marks 2 -> 1
Changed lines of the file:
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@@
   (junction (at 107.95 58.42) (diameter 0) (color 0 0 0 0)
   )
+  (junction (at 71.12 50.8) (diameter 0) (color 0 0 0 0)
+  )
   (junction (at 107.95 68.58) (diameter 0) (color 0 0 0 0)
   )
   (no_connect (at 102.87 50.8))
-  (no_connect (at 72.39 48.26))
   (wire (pts (xy 102.87 53.34) (xy 105.41 53.34))
     (stroke (width 0) (type default))
   )
+  (wire (pts (xy 71.12 48.26) (xy 71.12 50.8))
+    (stroke (width 0) (type default))
+  )
   (wire (pts (xy 242.57 48.26) (xy 242.57 52.07))
     (stroke (width 0) (type default))
@@
   )
   (wire (pts (xy 105.41 53.34) (xy 110.49 53.34))
+    (stroke (width 0) (type default))
+  )
+  (wire (pts (xy 72.39 48.26) (xy 71.12 48.26))
     (stroke (width 0) (type default))
   )
@@
       (effects (font (size 1.27 1.27)))
     )
-    (property "Value" "CCG30-24-12S_P" (at 87.63 43.18 0)
-      (effects (font (size 1.27 1.27)))
-    )
+    (property "Value" "CCG30-24-12S" (at 87.63 43.18 0)
+      (effects (font (size 1.27 1.27)))
+    )
