File: tsukuba_challenge.kicad_pcb (KiCad board)
At the start: 2 copper layers, 90 x 90 mm, 93 parts, among them IC1 ISOW1044BDFMR, J1 PWR_BATT, J10 CAN, J11 Relay, J12 EMS_SW, J13 EMS_SW, J14 Remote_SW, J15 Remote_SW, J2 USB_C_Receptacle_USB2.0_16P, J3 ST-LINK, J4 INDICATOR, J5 INDICATOR, J6 INDICATOR, J7 CAN, J8 CAN, J9 CAN, Q1 TBD62083AFWG_Z,EHZ, Q2 Q_NMOS_GDS, Q3 Q_PMOS_GSD, Q4 Q_NMOS_GSD, SW1 SPST_SW, U1 USBLC6-2SC6, U2 STM32F103CBTx, U3 L7805, U4 XC6206P332MR, Y1 12MHz

Commit message: 4/2(1)
Parts:
- added G***: LOGO, my_logo_pretty:rdclab_small, F.Cu at (73.0, 117.5)
- added REF**: KiCad-Logo2_5mm_SilkScreen, Symbol:KiCad-Logo2_5mm_SilkScreen, F.Cu at (94.8, 78.0)
- moved SW1 91.5 mm to (109.4, 78.5), turned to -90 degrees
- moved C9 84.1 mm to (108.2, 74.0)
- moved FB1 77.8 mm to (110.5, 90.0), turned to -90 degrees
- moved R9 75.7 mm to (109.5, 104.5), turned to -90 degrees
- moved D1 74.9 mm to (83.2, 114.5)
- moved C7 71.2 mm to (112.5, 90.2), turned to -90 degrees
- moved C8 70.6 mm to (114.0, 90.2), turned to -90 degrees
- moved R6 67.6 mm to (86.7, 114.5), turned to 180 degrees
- moved Q4 50.6 mm to (124.6, 78.5), turned to 180 degrees
- moved R18 47.1 mm to (120.7, 78.5)
- moved R5 42.9 mm to (100.8, 97.0)
- moved R20 42.6 mm to (125.5, 81.8), turned to -90 degrees
- moved R4 39.9 mm to (100.8, 98.5)
- moved R19 39.5 mm to (128.7, 79.5)
- moved R3 36.4 mm to (101.5, 101.0), turned to 90 degrees
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Routing:
- net +12V: track 0.00 -> 196.2 mm
- net +3.3V: track 0.00 -> 131.5 mm, vias 0 -> 2
- net +5V: track 0.00 -> 108.8 mm
- net /CAN_Transceiver/CAN_L: track 0.00 -> 72.7 mm
- net /CAN_Transceiver/CAN_H: track 0.00 -> 65.9 mm
- net +BATT: track 0.00 -> 47.6 mm
- net /STM32F103/INDICATOR_RED: track 0.00 -> 37.3 mm, vias 0 -> 2
- net /CAN_Transceiver/CAN_TX: track 0.00 -> 36.2 mm, vias 0 -> 2
- net /STM32F103/INDICATOR_YELLOW: track 0.00 -> 35.4 mm, vias 0 -> 2
- net /CAN_Transceiver/CAN_RX: track 0.00 -> 34.4 mm, vias 0 -> 2
- net /D-_OUT: track 0.00 -> 32.5 mm, vias 0 -> 2
- net /EMS/MCU_EMS_OBSERVE: track 0.00 -> 31.1 mm, vias 0 -> 2
- net Net-(J12-Pin_1): track 0.00 -> 30.9 mm
- net /MCU_CYCLE_LED: track 0.00 -> 30.7 mm, vias 0 -> 2
- net GND: track 0.00 -> 30.6 mm, vias 0 -> 124
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- added copper zone on B.Cu, net GND
- added copper zone on F.Cu, net GND
- added copper zone on B.Cu, net GNDPWR
- added copper zone on F.Cu, net GNDPWR
Other:
- board size 90 x 90 mm -> 90 x 70 mm
- board text added: "12V"
- board text added: "3.3V"
- board text added: "5V"
- board text added: "MCU"
- board text added: "遠隔スイッチ"
- board text added: "電源表示"
- board text added: "非常停"

Commit message: 4/2(2)
Parts:
- moved G*** 1.58 mm to (73.5, 119.0)
Routing:
- net GND: track 30.6 -> 32.1 mm
- net GNDPWR: vias 28 -> 30
Other:
- board text added: "ST-LINK"
- board text added: "リセット"
- board text added: "リレー"
- board text added: "ローバー主制御基板 Ver.0.1.0 設計：cmos"
- board text added: "上位"
- board text added: "表示灯"
- board text added: "電源"
- board text added: "駆動ESC"

Commit message: 🐛fix:
Parts:
- moved C16 5.52 mm to (90.5, 95.5)
- moved C14 2.28 mm to (90.0, 85.0)
- moved C12 2.01 mm to (88.8, 83.0)
- moved C15 0.25 mm to (90.0, 93.8)
- moved IC1 0.10 mm to (73.0, 102.0)
- moved Q3 0.08 mm to (126.6, 88.5)
- moved Q4 0.06 mm to (124.5, 78.6)
Routing:
- net +3.3V: track 131.5 -> 141.4 mm, vias 2 -> 4
- net +BATT: track 47.6 -> 38.5 mm
- net GND: track 32.1 -> 34.4 mm, vias 124 -> 123
- net +5V: track 108.8 -> 111.0 mm
- net +12V: track 196.2 -> 194.5 mm
- net GNDPWR: vias 30 -> 29

Commit message: 4/12
Parts:
- added JP3: EMS_Jumper, Connector_PinHeader_2.54mm:PinHeader_1x02_P2.54mm_Vertical, F.Cu at (127.0, 94.0)
- D1: value LED -> LED_MCU
- J2: value USB_C_Receptacle_USB2.0_16P -> USB_C_Receptacle_USB2.0
Routing:
- net Net-(J15-Pin_1): track 5.17 -> 11.3 mm
Changed lines of the file:
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@@
   (net 103 "unconnected-(U2-PB4-Pad40)")
   (net 104 "unconnected-(U2-PB7-Pad43)")
+  (footprint "Connector_PinHeader_2.54mm:PinHeader_1x02_P2.54mm_Vertical" (layer "F.Cu")
+    (at 127 94)
+    (descr "Through hole straight pin header, 1x02, 2.54mm pitch, single row")
+    (tags "Through hole pin header THT 1x02 2.54mm single row")
+    (property "Sheetfile" "EMS.kicad_sch")
+    (property "Sheetname" "EMS")
+    (property "ki_description" "Jumper, 2-pole, open")
+    (property "ki_keywords" "Jumper SPST")
+    (attr through_hole)
+    (fp_text reference "JP3" (at -3 0) (layer "F.SilkS")
+        (effects (font (size 1 1) (thickness 0.15)))
+    )
+    (fp_text value "EMS_Jumper" (at 0 4.87) (layer "F.Fab")
+        (effects (font (size 1 1) (thickness 0.15)))
+    )
+    (fp_text user "${REFERENCE}" (at 0 1.27 90) (layer "F.Fab")
+        (effects (font (size 1 1) (thickness 0.15)))
+    )
+    (fp_line (start -1.33 -1.33) (end 0 -1.33)
+      (stroke (width 0.12) (type solid)) (layer "F.SilkS"))
+    (fp_line (start -1.33 0) (end -1.33 -1.33)
+      (stroke (width 0.12) (type solid)) (layer "F.SilkS"))
+    (fp_line (start -1.33 1.27) (end -1.33 3.87)
+      (stroke (width 0.12) (type solid)) (layer "F.SilkS"))
+    (fp_line (start -1.33 1.27) (end 1.33 1.27)
+      (stroke (width 0.12) (type solid)) (layer "F.SilkS"))
+    (fp_line (start -1.33 3.87) (end 1.33 3.87)
+      (stroke (width 0.12) (type solid)) (layer "F.SilkS"))
+    (fp_line (start 1.33 1.27) (end 1.33 3.87)
+      (stroke (width 0.12) (type solid)) (layer "F.SilkS"))
+    (fp_line (start -1.8 -1.8) (end -1.8 4.35)
+      (stroke (width 0.05) (type solid)) (layer "F.CrtYd"))
+    (fp_line (start -1.8 4.35) (end 1.8 4.35)
+      (stroke (width 0.05) (type solid)) (layer "F.CrtYd"))
+    (fp_line (start 1.8 -1.8) (end -1.8 -1.8)
+      (stroke (width 0.05) (type solid)) (layer "F.CrtYd"))
+    (fp_line (start 1.8 4.35) (end 1.8 -1.8)
+      (stroke (width 0.05) (type solid)) (layer "F.CrtYd"))
+    (fp_line (start -1.27 -0.635) (end -0.635 -1.27)
+      (stroke (width 0.1) (type solid)) (layer "F.Fab"))
+    (fp_line (start -1.27 3.81) (end -1.27 -0.635)
+      (stroke (width 0.1) (type solid)) (layer "F.Fab"))
+    (fp_line (start -0.635 -1.27) (end 1.27 -1.27)
+      (stroke (width 0.1) (type solid)) (layer "F.Fab"))
+    (fp_line (start 1.27 -1.27) (end 1.27 3.81)
+      (stroke (width 0.1) (type solid)) (layer "F.Fab"))
+    (fp_line (start 1.27 3.81) (end -1.27 3.81)
+      (stroke (width 0.1) (type solid)) (layer "F.Fab"))
+    (pad "1" thru_hole rect (at 0 0) (size 1.7 1.7) (drill 1) (layers "*.Cu" "*.Mask")
+      (net 58 "Net-(J15-Pin_1)") (pinfunction "A") (pintype "passive"))
+    (pad "2" thru_hole oval (at 0 2.54) (size 1.7 1.7) (drill 1) (layers "*.Cu" "*.Mask")
+      (net 1 "GND") (pinfunction "B") (pintype "passive"))
+    (model "${KICAD6_3DMODEL_DIR}/Connector_PinHeader_2.54mm.3dshapes/PinHeader_1x02_P2.54mm_Vertical.wrl"
+      (offset (xyz 0 0 0))
+      (scale (xyz 1 1 1))
+      (rotate (xyz 0 0 0))
+    )
+  )
   (footprint "Capacitor_SMD:C_0603_1608Metric" (layer "F.Cu")
     (at 120 105 180)
@@
         (effects (font (size 1 1) (thickness 0.15)))
     )
-    (fp_text value "MountingHole" (at 0 4.2) (layer "F.Fab") hide
+    (fp_text value "MountingHole" (at 0 4.2) (layer "F.Fab")
         (effects (font (size 1 1) (thickness 0.15)))
     )
@@
         (effects (font (size 1 1) (thickness 0.15)))
     )
-    (fp_text value "MountingHole" (at 0 4.2) (layer "F.Fab") hide
+    (fp_text value "MountingHole" (at 0 4.2) (layer "F.Fab")
         (effects (font (size 1 1) (thickness 0.15)))
     )
@@
     (property "Sheetfile" "tsukuba_challenge.kicad_sch")
     (property "Sheetname" "")
-    (property "ki_description" "USB 2.0-only 16P Type-C Receptacle connector")
+    (property "ki_description" "USB 2.0-only Type-C Receptacle connector")
     (property "ki_keywords" "usb universal serial bus type-C USB2.0")
     (attr smd)
@@
         (effects (font (size 1 1) (thickness 0.15)))
     )
-    (fp_text value "USB_C_Receptacle_USB2.0_16P" (at 0 5) (layer "F.Fab") hide
+    (fp_text value "USB_C_Receptacle_USB2.0" (at 0 5) (layer "F.Fab") hide
         (effects (font (size 1 1) (thickness 0.15)))
     )
@@
         (effects (font (size 1 1) (thickness 0.15)))
     )
-    (fp_text value "MountingHole" (at 0 4.2) (layer "F.Fab") hide
+    (fp_text value "MountingHole" (at 0 4.2) (layer "F.Fab")
         (effects (font (size 1 1) (thickness 0.15)))
     )
@@
     (fp_line (start 4.11 2.7) (end 3.11 2.7)
       (stroke (width 0.1) (type solid)) (layer "F.Fab"))
-    (pad "1" smd roundrect (at -5.04 -2.28) (size 2.2 1.2) (layers "F.Cu" "F.Paste" "F.Mask") (roundrect_rratio 0.208333)
+    (pad "1" smd roundrect (at -5.04 -2.28) (size 2.2 1.2) (layers "F.Cu" "F.Paste" "F.Mask") (roundrect_rratio 0.2083333333)
       (net 8 "+12V") (pinfunction "IN") (pintype "power_in"))
-    (pad "2" smd roundrect (at -0.415 -1.525) (size 3.05 2.75) (layers "F.Cu" "F.Paste") (roundrect_rratio 0.090909)
+    (pad "2" smd roundrect (at -0.415 -1.525) (size 3.05 2.75) (layers "F.Cu" "F.Paste") (roundrect_rratio 0.09090909091)
       (net 1 "GND") (pinfunction "GND") (pintype "power_in"))
-    (pad "2" smd roundrect (at -0.415 1.525) (size 3.05 2.75) (layers "F.Cu" "F.Paste") (roundrect_rratio 0.090909)
+    (pad "2" smd roundrect (at -0.415 1.525) (size 3.05 2.75) (layers "F.Cu" "F.Paste") (roundrect_rratio 0.09090909091)
       (net 1 "GND") (pinfunction "GND") (pintype "power_in"))
-    (pad "2" smd roundrect (at 1.26 0) (size 6.4 5.8) (layers "F.Cu" "F.Mask") (roundrect_rratio 0.043103)
+    (pad "2" smd roundrect (at 1.26 0) (size 6.4 5.8) (layers "F.Cu" "F.Mask") (roundrect_rratio 0.04310293103)
       (net 1 "GND") (pinfunction "GND") (pintype "power_in"))
-    (pad "2" smd roundrect (at 2.935 -1.525) (size 3.05 2.75) (layers "F.Cu" "F.Paste") (roundrect_rratio 0.090909)
+    (pad "2" smd roundrect (at 2.935 -1.525) (size 3.05 2.75) (layers "F.Cu" "F.Paste") (roundrect_rratio 0.09090909091)
       (net 1 "GND") (pinfunction "GND") (pintype "power_in"))
-    (pad "2" smd roundrect (at 2.935 1.525) (size 3.05 2.75) (layers "F.Cu" "F.Paste") (roundrect_rratio 0.090909)
+    (pad "2" smd roundrect (at 2.935 1.525) (size 3.05 2.75) (layers "F.Cu" "F.Paste") (roundrect_rratio 0.09090909091)
       (net 1 "GND") (pinfunction "GND") (pintype "power_in"))
-    (pad "3" smd roundrect (at -5.04 2.28) (size 2.2 1.2) (layers "F.Cu" "F.Paste" "F.Mask") (roundrect_rratio 0.208333)
+    (pad "3" smd roundrect (at -5.04 2.28) (size 2.2 1.2) (layers "F.Cu" "F.Paste" "F.Mask") (roundrect_rratio 0.2083333333)
       (net 2 "+5V") (pinfunction "OUT") (pintype "power_out"))
     (model "${KICAD6_3DMODEL_DIR}/Package_TO_SOT_SMD.3dshapes/TO-252-2.wrl"
@@
         (effects (font (size 1 1) (thickness 0.15)))
     )
-    (fp_text value "LED" (at 0 1.43) (layer "F.Fab")
+    (fp_text value "LED_MCU" (at 0 1.43) (layer "F.Fab")
         (effects (font (size 1 1) (thickness 0.15)))
     )
@@
         (effects (font (size 1 1) (thickness 0.15)))
     )
-    (fp_text value "MountingHole" (at 0 4.2) (layer "F.Fab") hide
+    (fp_text value "MountingHole" (at 0 4.2) (layer "F.Fab")
         (effects (font (size 1 1) (thickness 0.15)))
     )
@@
   (segment (start 129.825 71) (end 127.825 73) (width 0.25) (layer "F.Cu") (net 56))
   (segment (start 131 89.5) (end 135.58 89.5) (width 0.25) (layer "F.Cu") (net 58))
+  (segment (start 131 89.5) (end 131 90) (width 0.25) (layer "F.Cu") (net 58))
   (segment (start 135.58 89.5) (end 136 89.08) (width 0.25) (layer "F.Cu") (net 58))
+  (segment (start 131 90) (end 127 94) (width 0.25) (layer "F.Cu") (net 58))
   (segment (start 90 70.805) (end 89.92 70.725) (width 0.25) (layer "F.Cu") (net 61))
   (segment (start 90 72.5) (end 90 70.805) (width 0.25) (layer "F.Cu") (net 61))

Commit message: 4/12
Parts:
- C13: value 120u -> 100u
Changed lines of the file:
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@@
     (descr "SMD capacitor, aluminum electrolytic, Nichicon, 6.3x7.7mm")
     (tags "capacitor electrolytic")
+    (property "LCSC" "C5355875")
     (property "Sheetfile" "power.kicad_sch")
     (property "Sheetname" "Power")
@@
         (effects (font (size 1 1) (thickness 0.15)))
     )
-    (fp_text value "120u" (at 0 4.35 90) (layer "F.Fab")
+    (fp_text value "100u" (at 0 4.35 90) (layer "F.Fab")
         (effects (font (size 1 1) (thickness 0.15)))
     )

Commit message: 4/13 product update
Parts:
- D5: footprint Diode_SMD:D_SMA -> my_pretty:SOD-123FL
- moved D5 0.13 mm to (119.0, 62.1), turned to 90 degrees
Routing:
- net GND: vias 123 -> 124

Commit message: product data
Parts:
- C12: footprint Capacitor_SMD:C_0603_1608Metric -> Capacitor_SMD:C_1206_3216Metric
- moved C12 1.22 mm to (90.0, 83.0)
Routing:
- net GND: track 34.4 -> 36.8 mm, vias 124 -> 125
Changed lines of the file:
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@@
     )
   )
-  (footprint "Capacitor_SMD:C_0603_1608Metric" (layer "F.Cu")
-    (at 88.775 83)
-    (descr "Capacitor SMD 0603 (1608 Metric), square (rectangular) end terminal, IPC_7351 nominal, (Body size source: IPC-SM-782 page 76, https://www.pcb-3d.com/wordpress/wp-content/uploads/ipc-sm-782a_amendment_1_and_2.pdf), generated with kicad-footprint-generator")
+  (footprint "Capacitor_SMD:C_1206_3216Metric" (layer "F.Cu")
+    (at 90 83)
+    (descr "Capacitor SMD 1206 (3216 Metric), square (rectangular) end terminal, IPC_7351 nominal, (Body size source: IPC-SM-782 page 76, https://www.pcb-3d.com/wordpress/wp-content/uploads/ipc-sm-782a_amendment_1_and_2.pdf), generated with kicad-footprint-generator")
     (tags "capacitor")
+    (property "LCSC" "C12891")
     (property "Sheetfile" "power.kicad_sch")
     (property "Sheetname" "Power")
@@
     (property "ki_keywords" "capacitor cap")
     (attr smd)
-    (fp_text reference "C12" (at 2.725 0) (layer "F.SilkS")
-        (effects (font (size 1 1) (thickness 0.15)))
-    )
-    (fp_text value "22u" (at 0 1.43) (layer "F.Fab")
+    (fp_text reference "C12" (at 3.5 0) (layer "F.SilkS")
+        (effects (font (size 1 1) (thickness 0.15)))
+    )
+    (fp_text value "22u" (at 0 1.85) (layer "F.Fab")
         (effects (font (size 1 1) (thickness 0.15)))
     )
     (fp_text user "${REFERENCE}" (at 0 0) (layer "F.Fab")
-        (effects (font (size 0.4 0.4) (thickness 0.06)))
-    )
-    (fp_line (start -0.14058 -0.51) (end 0.14058 -0.51)
-      (stroke (width 0.12) (type solid)) (layer "F.SilkS"))
-    (fp_line (start -0.14058 0.51) (end 0.14058 0.51)
-      (stroke (width 0.12) (type solid)) (layer "F.SilkS"))
-    (fp_line (start -1.48 -0.73) (end 1.48 -0.73)
-      (stroke (width 0.05) (type solid)) (layer "F.CrtYd"))
-    (fp_line (start -1.48 0.73) (end -1.48 -0.73)
-      (stroke (width 0.05) (type solid)) (layer "F.CrtYd"))
-    (fp_line (start 1.48 -0.73) (end 1.48 0.73)
-      (stroke (width 0.05) (type solid)) (layer "F.CrtYd"))
-    (fp_line (start 1.48 0.73) (end -1.48 0.73)
-      (stroke (width 0.05) (type solid)) (layer "F.CrtYd"))
-    (fp_line (start -0.8 -0.4) (end 0.8 -0.4)
-      (stroke (width 0.1) (type solid)) (layer "F.Fab"))
-    (fp_line (start -0.8 0.4) (end -0.8 -0.4)
-      (stroke (width 0.1) (type solid)) (layer "F.Fab"))
-    (fp_line (start 0.8 -0.4) (end 0.8 0.4)
-      (stroke (width 0.1) (type solid)) (layer "F.Fab"))
-    (fp_line (start 0.8 0.4) (end -0.8 0.4)
-      (stroke (width 0.1) (type solid)) (layer "F.Fab"))
-    (pad "1" smd roundrect (at -0.775 0) (size 0.9 0.95) (layers "F.Cu" "F.Paste" "F.Mask") (roundrect_rratio 0.25)
+        (effects (font (size 0.8 0.8) (thickness 0.12)))
+    )
+    (fp_line (start -0.711252 -0.91) (end 0.711252 -0.91)
+      (stroke (width 0.12) (type solid)) (layer "F.SilkS"))
+    (fp_line (start -0.711252 0.91) (end 0.711252 0.91)
+      (stroke (width 0.12) (type solid)) (layer "F.SilkS"))
+    (fp_line (start -2.3 -1.15) (end 2.3 -1.15)
+      (stroke (width 0.05) (type solid)) (layer "F.CrtYd"))
+    (fp_line (start -2.3 1.15) (end -2.3 -1.15)
+      (stroke (width 0.05) (type solid)) (layer "F.CrtYd"))
+    (fp_line (start 2.3 -1.15) (end 2.3 1.15)
+      (stroke (width 0.05) (type solid)) (layer "F.CrtYd"))
+    (fp_line (start 2.3 1.15) (end -2.3 1.15)
+      (stroke (width 0.05) (type solid)) (layer "F.CrtYd"))
+    (fp_line (start -1.6 -0.8) (end 1.6 -0.8)
+      (stroke (width 0.1) (type solid)) (layer "F.Fab"))
+    (fp_line (start -1.6 0.8) (end -1.6 -0.8)
+      (stroke (width 0.1) (type solid)) (layer "F.Fab"))
+    (fp_line (start 1.6 -0.8) (end 1.6 0.8)
+      (stroke (width 0.1) (type solid)) (layer "F.Fab"))
+    (fp_line (start 1.6 0.8) (end -1.6 0.8)
+      (stroke (width 0.1) (type solid)) (layer "F.Fab"))
+    (pad "1" smd roundrect (at -1.475 0) (size 1.15 1.8) (layers "F.Cu" "F.Paste" "F.Mask") (roundrect_rratio 0.2173913043)
       (net 8 "+12V") (pintype "passive"))
-    (pad "2" smd roundrect (at 0.775 0) (size 0.9 0.95) (layers "F.Cu" "F.Paste" "F.Mask") (roundrect_rratio 0.25)
+    (pad "2" smd roundrect (at 1.475 0) (size 1.15 1.8) (layers "F.Cu" "F.Paste" "F.Mask") (roundrect_rratio 0.2173913043)
       (net 1 "GND") (pintype "passive"))
-    (model "${KICAD6_3DMODEL_DIR}/Capacitor_SMD.3dshapes/C_0603_1608Metric.wrl"
+    (model "${KICAD6_3DMODEL_DIR}/Capacitor_SMD.3dshapes/C_1206_3216Metric.wrl"
       (offset (xyz 0 0 0))
       (scale (xyz 1 1 1))
@@
   )
   (segment (start 115.725 101.725) (end 115.75 101.75) (width 0.25) (layer "F.Cu") (net 1))
+  (segment (start 91.275 84.5) (end 93 84.5) (width 0.5) (layer "F.Cu") (net 1))
   (segment (start 103.75 102.55) (end 104.5 102.55) (width 0.25) (layer "F.Cu") (net 1))
   (segment (start 106.75 91.984314) (end 107.234314 91.5) (width 0.25) (layer "F.Cu") (net 1))
@@
   (segment (start 92.2 102.45) (end 92.25 102.5) (width 0.5) (layer "F.Cu") (net 1))
   (segment (start 104.034314 99.2) (end 103.2 100.034314) (width 0.25) (layer "F.Cu") (net 1))
+  (segment (start 90.775 85) (end 91.275 84.5) (width 0.5) (layer "F.Cu") (net 1))
   (segment (start 103.2 102) (end 103.75 102.55) (width 0.25) (layer "F.Cu") (net 1))
   (segment (start 117.2125 108.2875) (end 116.5 109) (width 0.25) (layer "F.Cu") (net 1))
@@
   (via (at 96.75 74.25) (size 0.8) (drill 0.4) (layers "F.Cu" "B.Cu") (free) (net 1))
   (via (at 117 115.75) (size 0.8) (drill 0.4) (layers "F.Cu" "B.Cu") (free) (net 1))
+  (via (at 88.5 81) (size 0.8) (drill 0.4) (layers "F.Cu" "B.Cu") (free) (net 1))
   (via (at 104.5 92.5) (size 0.8) (drill 0.4) (layers "F.Cu" "B.Cu") (free) (net 1))
   (via (at 104.5 109.5) (size 0.3) (drill 0.15) (layers "F.Cu" "B.Cu") (net 1))
@@
   (via (at 96.25 99.5) (size 0.8) (drill 0.4) (layers "F.Cu" "B.Cu") (free) (net 1))
   (via (at 137 106.5) (size 0.8) (drill 0.4) (layers "F.Cu" "B.Cu") (free) (net 1))
-  (via (at 88.75 81.5) (size 0.8) (drill 0.4) (layers "F.Cu" "B.Cu") (free) (net 1))
   (via (at 83.25 117.75) (size 0.8) (drill 0.4) (layers "F.Cu" "B.Cu") (free) (net 1))
   (via (at 88 56.5) (size 0.8) (drill 0.4) (layers "F.Cu" "B.Cu") (free) (net 1))
@@
   (via (at 139.25 99) (size 0.8) (drill 0.4) (layers "F.Cu" "B.Cu") (free) (net 1))
   (via (at 120.25 54) (size 0.8) (drill 0.4) (layers "F.Cu" "B.Cu") (free) (net 1))
+  (via (at 88.5 75) (size 0.8) (drill 0.4) (layers "F.Cu" "B.Cu") (free) (net 1))
   (via (at 77.5 85.25) (size 0.8) (drill 0.4) (layers "F.Cu" "B.Cu") (free) (net 1))
   (via (at 131.25 62.75) (size 0.8) (drill 0.4) (layers "F.Cu" "B.Cu") (free) (net 1))
@@
   (segment (start 117.35 100.175) (end 117.275 100.25) (width 0.25) (layer "F.Cu") (net 7))
   (segment (start 113.1625 97.7) (end 114.54038 97.7) (width 0.25) (layer "F.Cu") (net 7))
+  (segment (start 88.525 83) (end 85.85 83) (width 0.5) (layer "F.Cu") (net 8))
   (segment (start 127.25 52.25) (end 125.25 52.25) (width 0.5) (layer "F.Cu") (net 8))
   (segment (start 80.5 59.5) (end 80.5 81.97) (width 1) (layer "F.Cu") (net 8))
@@
   (segment (start 130.632538 84) (end 133.5 84) (width 0.25) (layer "F.Cu") (net 8))
   (segment (start 89.225 85) (end 89.225 86.995) (width 0.5) (layer "F.Cu") (net 8))
-  (segment (start 83.69 85.16) (end 85.85 83) (width 0.5) (layer "F.Cu") (net 8))
   (segment (start 127.25 52.25) (end 130.5 55.5) (width 0.5) (layer "F.Cu") (net 8))
   (segment (start 137.5 62) (end 139 63.5) (width 0.5) (layer "F.Cu") (net 8))
   (segment (start 112.5 57) (end 115.5 57) (width 0.25) (layer "F.Cu") (net 8))
-  (segment (start 88 83.775) (end 89.225 85) (width 0.5) (layer "F.Cu") (net 8))
   (segment (start 100.933604 52.05) (end 101.5 52.05) (width 0.5) (layer "F.Cu") (net 8))
   (segment (start 107.5 66.1) (end 107.5 62) (width 0.25) (layer "F.Cu") (net 8))
@@
   (segment (start 123.5 54) (end 123.5 56) (width 0.5) (layer "F.Cu") (net 8))
   (segment (start 115.5 57) (end 118.5 54) (width 0.25) (layer "F.Cu") (net 8))
-  (segment (start 88 83) (end 88 83.775) (width 0.5) (layer "F.Cu") (net 8))
-  (segment (start 85.85 83) (end 88 83) (width 0.5) (layer "F.Cu") (net 8))
+  (segment (start 85.85 83) (end 83.69 85.16) (width 0.5) (layer "F.Cu") (net 8))
   (segment (start 130.5 58.5) (end 134 62) (width 0.5) (layer "F.Cu") (net 8))
   (segment (start 136 84) (end 133.5 84) (width 0.25) (layer "F.Cu") (net 8))
@@
   (segment (start 89.225 86.995) (end 89.425 87.195) (width 0.5) (layer "F.Cu") (net 8))
   (segment (start 80.5 81.97) (end 83.69 85.16) (width 1) (layer "F.Cu") (net 8))
+  (segment (start 88.525 84.3) (end 89.225 85) (width 0.5) (layer "F.Cu") (net 8))
   (segment (start 117.775 61.225) (end 118.5 60.5) (width 0.25) (layer "F.Cu") (net 8))
   (segment (start 87.95 52.05) (end 101.5 52.05) (width 0.5) (layer "F.Cu") (net 8))
@@
   (segment (start 118.5 60.5) (end 119 60.5) (width 0.25) (layer "F.Cu") (net 8))
   (segment (start 101.5 52.05) (end 118.5 52.05) (width 0.5) (layer "F.Cu") (net 8))
+  (segment (start 88.525 83) (end 88.525 84.3) (width 0.5) (layer "F.Cu") (net 8))
   (segment (start 118.5 52.05) (end 121.55 52.05) (width 0.5) (layer "F.Cu") (net 8))
   (segment (start 55 68.9) (end 55 70.65) (width 1) (layer "F.Cu") (net 9))
@@
     (polygon
       (pts
-        (xy 88.25 85)
-        (xy 92.25 85)
+        (xy 88.25 84)
+        (xy 92.25 84)
         (xy 92.25 92.5)
         (xy 88.25 92.5)
