File: tsukuba_challenge.kicad_pcb (KiCad board)
At the start: 2 copper layers, 90 x 70 mm, 96 parts, among them IC1 ISOW1044BDFMR, J1 PWR_BATT, J10 CAN, J11 Relay, J12 EMS_SW, J13 EMS_SW, J14 Remote_SW, J15 Remote_SW, J2 USB_C_Receptacle_USB2.0, J3 ST-LINK, J4 INDICATOR, J5 INDICATOR, J6 INDICATOR, J7 CAN, J8 CAN, J9 CAN, Q1 TBD62083AFWG_Z,EHZ, Q2 Q_NMOS_GDS, Q3 Q_PMOS_GSD, Q4 Q_NMOS_GSD, SW1 SPST_SW, U1 USBLC6-2SC6, U2 STM32F103CBTx, U3 L7805, U4 XC6206P332MR, Y1 12MHz

Commit message: ✨feat:f302
Parts:
- H1, H2, H3, H4: footprint MountingHole:MountingHole_3.2mm_M3 -> MountingHole:MountingHole_4.3mm_M4
- PS1: value CCG30-24-12S_P -> CCG30-24-12S
- Q2: value Q_NMOS_GDS -> Q_NMOS_GSD
- R4: value 22 -> 33k
- R5: value 22 -> 82k
- U2: value STM32F103CBTx -> STM32F302CBTx
- moved R3 3.29 mm to (100.0, 98.1)
- moved R5 3.07 mm to (98.2, 95.3), turned to -90 degrees
- moved R4 2.58 mm to (98.2, 98.7), turned to 90 degrees
- moved U1 1.75 mm to (119.0, 106.4)
- moved C1 1.50 mm to (120.0, 103.5)
- moved Q2 0.12 mm to (124.0, 67.9), turned to 90 degrees
Connections:
- net /STM32F103/INDICATOR_BUZZER renamed /STM32F302/INDICATOR_BUZZER
- net /STM32F103/INDICATOR_GREEN renamed /STM32F302/INDICATOR_GREEN
- net /STM32F103/INDICATOR_RED renamed /STM32F302/INDICATOR_RED
- net /STM32F103/INDICATOR_YELLOW renamed /STM32F302/INDICATOR_YELLOW
- net /STM32F103/SWCLK renamed /STM32F302/SWCLK
- net /STM32F103/SWDIO renamed /STM32F302/SWDIO
- net /STM32F103/SWO renamed /STM32F302/SWO
- J2 pad A4: unconnected-(J2-VBUS-PadA4) -> /USB_VBUS
- J2 pad A9: unconnected-(J2-VBUS-PadA4) -> /USB_VBUS
- J2 pad B4: unconnected-(J2-VBUS-PadA4) -> /USB_VBUS
- J2 pad B9: unconnected-(J2-VBUS-PadA4) -> /USB_VBUS
- PS1 pad 1: unconnected-(PS1-RC-Pad1) -> GNDPWR
- Q2 pad 2: Net-(D6-K) -> GND
- Q2 pad 3: GND -> Net-(D6-K)
- R3 pad 1: +3.3V -> /D+_OUT
- R3 pad 2: /STM32F103/USB_D+ -> /STM32F302/USB_PULLUP
- R4 pad 1: /D+_OUT -> /USB_VBUS
- R4 pad 2: /STM32F103/USB_D+ -> /STM32F302/USB_VBUS
- R5 pad 1: /D-_OUT -> GND
- R5 pad 2: /STM32F103/USB_D- -> /STM32F302/USB_VBUS
- U2 pad 30: unconnected-(U2-PA9-Pad30) -> /STM32F302/USB_VBUS
- U2 pad 31: unconnected-(U2-PA10-Pad31) -> /STM32F302/USB_PULLUP
- U2 pad 32: /STM32F103/USB_D- -> /D-_OUT
- U2 pad 33: /STM32F103/USB_D+ -> /D+_OUT
Routing:
- net /USB_VBUS: track 0.00 -> 43.0 mm, vias 0 -> 3
- net /D+_OUT: track 25.2 -> 34.5 mm
- net /STM32F302/USB_VBUS: track 0.00 -> 8.49 mm
- net /STM32F103/USB_D+: track 5.05 -> 0.00 mm
- net /STM32F302/USB_PULLUP: track 0.00 -> 4.86 mm
- net /D+_IN: track 12.9 -> 17.0 mm
- net GND: track 36.8 -> 32.8 mm, vias 125 -> 124
- net +3.3V: track 141.4 -> 137.5 mm
- net /STM32F103/USB_D-: track 3.48 -> 0.00 mm
- net +5V: track 111.0 -> 107.9 mm
- net /D-_IN: track 8.30 -> 11.3 mm
- net Net-(J2-CC2): track 6.02 -> 7.73 mm
- net /CAN_Transceiver/CAN_TX: track 36.2 -> 37.2 mm
- net /D-_OUT: track 32.5 -> 31.6 mm
- net Net-(J2-CC1): track 9.69 -> 10.6 mm
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