File: tsukuba_challenge.kicad_pcb (KiCad board)
At the start: 2 copper layers, 90 x 70 mm, 96 parts, among them IC1 ISOW1044BDFMR, J1 PWR_BATT, J10 CAN, J11 Relay, J12 EMS_SW, J13 EMS_SW, J14 Remote_SW, J15 Remote_SW, J2 USB_C_Receptacle_USB2.0, J3 ST-LINK, J4 INDICATOR, J5 INDICATOR, J6 INDICATOR, J7 CAN, J8 CAN, J9 CAN, Q1 TBD62083AFWG_Z,EHZ, Q2 Q_NMOS_GSD, Q3 Q_PMOS_GSD, Q4 Q_NMOS_GSD, SW1 SPST_SW, U1 USBLC6-2SC6, U2 STM32F302CBTx, U3 L7805, U4 XC6206P332MR, Y1 12MHz

Commit message: 6/29
Parts:
- C14: value 0.33u -> 0.47u
- moved R9 5.65 mm to (109.5, 110.2)
- moved C1 1.40 mm to (120.0, 104.9)
- moved U1 0.97 mm to (119.2, 107.3), turned to 180 degrees
Connections:
- U1 pad 1: /D+_IN -> /D-_IN
- U1 pad 3: /D-_IN -> /D+_IN
- U1 pad 4: /D-_OUT -> /D+_OUT
- U1 pad 6: /D+_OUT -> /D-_OUT
- U2 pad 12: unconnected-(U2-PA2-Pad12) -> /EMS/MCU_EMS_OBSERVE
- U2 pad 21: /STM32F302/INDICATOR_RED -> unconnected-(U2-PB10-Pad21)
- U2 pad 22: /STM32F302/INDICATOR_YELLOW -> unconnected-(U2-PB11-Pad22)
- U2 pad 25: /STM32F302/INDICATOR_GREEN -> /STM32F302/INDICATOR_BUZZER
- U2 pad 26: /STM32F302/INDICATOR_BUZZER -> /STM32F302/INDICATOR_GREEN
- U2 pad 27: unconnected-(U2-PB14-Pad27) -> /STM32F302/INDICATOR_YELLOW
- U2 pad 28: unconnected-(U2-PB15-Pad28) -> /STM32F302/INDICATOR_RED
- U2 pad 41: /EMS/MCU_EMS_OBSERVE -> unconnected-(U2-PB5-Pad41)
Routing:
- net GND: track 32.8 -> 21.7 mm, vias 124 -> 140
- net /EMS/MCU_EMS_OBSERVE: track 30.9 -> 21.3 mm, vias 2 -> 0
- net /MCU_CYCLE_LED: track 30.7 -> 39.5 mm
- net /USB_VBUS: track 43.0 -> 34.9 mm, vias 3 -> 2
- net +5V: track 107.9 -> 115.7 mm, vias 0 -> 4
- net /D+_IN: track 17.0 -> 9.86 mm, vias 4 -> 0
- net Net-(U2-BOOT0): track 2.72 -> 8.58 mm, vias 0 -> 2
- net +3.3V: track 137.5 -> 131.8 mm
- net /D-_IN: track 11.3 -> 6.26 mm
- net /STM32F302/INDICATOR_RED: track 37.3 -> 32.4 mm
- net /STM32F302/INDICATOR_YELLOW: track 35.5 -> 31.0 mm
- net /D-_OUT: track 31.6 -> 28.7 mm, vias 2 -> 0
- net /D+_OUT: track 34.5 -> 32.5 mm
- net /CAN_Transceiver/CAN_TX: track 37.2 -> 35.7 mm
- net Net-(SW1-B): track 27.5 -> 26.5 mm
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Other:
- board text added: "ローバー主制御基板 Ver.0.2 設計：cmos"
- board text removed: "ローバー主制御基板 Ver.0.1.0 設計：cmos"

Commit message: 7/19
Connections:
- J6 pad 1: unconnected-(J6-Pin_1-Pad1) -> GND
Routing:
- net GNDPWR: vias 34 -> 38
- net GND: vias 140 -> 146
Other:
- board text added: "ローバー主制御基板 Ver.0.3 設計：cmos"
- board text removed: "ローバー主制御基板 Ver.0.2 設計：cmos"
