File: CAN_Transceiver.kicad_sch (KiCad schematic)
At the start: 16 parts, among them IC1 ISOW1044BDFMR

Commit message: 4/2
Parts:
- C7: value 0.1uF -> 0.1u
- C9: value 10uF -> 10u
- IC1: footprint SOIC127P1030X355-20N -> Package_SO:SOIC-20W_7.5x12.8mm_P1.27mm
- R3: footprint Resistor_SMD:R_0805_2012Metric -> Resistor_SMD:R_0603_1608Metric
Connections:
- no-connect marks 2 -> 1
Changed lines of the file:
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@@
   )
   (no_connect (at 158.75 82.55))
-  (no_connect (at 123.19 82.55))
   (wire (pts (xy 161.29 102.87) (xy 172.72 102.87))
     (stroke (width 0) (type default))
@@
       (project "tsukuba_challenge"
         (path "/55f88ae9-9831-47be-a185-734020e38c84/9c1fd94d-8d77-4c45-be6e-46f605b5b044"
-          (reference "#PWR043") (unit 1)
+          (reference "#PWR045") (unit 1)
         )
       )
@@
       (project "tsukuba_challenge"
         (path "/55f88ae9-9831-47be-a185-734020e38c84/9c1fd94d-8d77-4c45-be6e-46f605b5b044"
-          (reference "FB1") (unit 1)
+          (reference "FB2") (unit 1)
         )
       )
@@
       (effects (font (size 1.27 1.27)) (justify left))
     )
-    (property "Value" "0.1uF" (at 162.56 59.69 0)
+    (property "Value" "0.1u" (at 162.56 59.69 0)
       (effects (font (size 1.27 1.27)) (justify left))
     )
@@
       (project "tsukuba_challenge"
         (path "/55f88ae9-9831-47be-a185-734020e38c84/9c1fd94d-8d77-4c45-be6e-46f605b5b044"
-          (reference "FB2") (unit 1)
+          (reference "FB3") (unit 1)
         )
       )
@@
       (effects (font (size 1.27 1.27)) (justify left))
     )
-    (property "Value" "10uF" (at 171.45 59.69 0)
+    (property "Value" "10u" (at 171.45 59.69 0)
       (effects (font (size 1.27 1.27)) (justify left))
     )
@@
   (symbol (lib_id "power:GNDPWR") (at 168.91 80.01 0) (unit 1)
     (in_bom yes) (on_board yes) (dnp no) (fields_autoplaced)
-    (property "Reference" "#PWR042" (at 168.91 85.09 0)
+    (property "Reference" "#PWR044" (at 168.91 85.09 0)
       (effects (font (size 1.27 1.27)) hide)
     )
@@
       (project "tsukuba_challenge"
         (path "/55f88ae9-9831-47be-a185-734020e38c84/9c1fd94d-8d77-4c45-be6e-46f605b5b044"
-          (reference "#PWR042") (unit 1)
+          (reference "#PWR044") (unit 1)
         )
       )
@@
       (project "tsukuba_challenge"
         (path "/55f88ae9-9831-47be-a185-734020e38c84/9c1fd94d-8d77-4c45-be6e-46f605b5b044"
-          (reference "#PWR041") (unit 1)
+          (reference "#PWR043") (unit 1)
         )
       )
@@
       (project "tsukuba_challenge"
         (path "/55f88ae9-9831-47be-a185-734020e38c84/9c1fd94d-8d77-4c45-be6e-46f605b5b044"
-          (reference "FB4") (unit 1)
+          (reference "FB5") (unit 1)
         )
       )
@@
       (project "tsukuba_challenge"
         (path "/55f88ae9-9831-47be-a185-734020e38c84/9c1fd94d-8d77-4c45-be6e-46f605b5b044"
-          (reference "FB5") (unit 1)
+          (reference "FB6") (unit 1)
         )
       )
@@
       (effects (font (size 1.27 1.27)))
     )
-    (property "Footprint" "SOIC127P1030X355-20N" (at 154.94 162.23 0)
+    (property "Footprint" "Package_SO:SOIC-20W_7.5x12.8mm_P1.27mm" (at 154.94 162.23 0)
       (effects (font (size 1.27 1.27)) (justify left top) hide)
     )
@@
       (project "tsukuba_challenge"
         (path "/55f88ae9-9831-47be-a185-734020e38c84/9c1fd94d-8d77-4c45-be6e-46f605b5b044"
-          (reference "FB3") (unit 1)
+          (reference "FB4") (unit 1)
         )
       )
@@
       (effects (font (size 1.27 1.27)) (justify left))
     )
-    (property "Footprint" "Resistor_SMD:R_0805_2012Metric" (at 95.758 63.5 90)
+    (property "Footprint" "Resistor_SMD:R_0603_1608Metric" (at 95.758 63.5 90)
       (effects (font (size 1.27 1.27)) hide)
     )
@@
       (project "tsukuba_challenge"
         (path "/55f88ae9-9831-47be-a185-734020e38c84/9c1fd94d-8d77-4c45-be6e-46f605b5b044"
-          (reference "R17") (unit 1)
+          (reference "R21") (unit 1)
         )
       )
@@
   (symbol (lib_id "power:GNDPWR") (at 204.47 113.03 0) (unit 1)
     (in_bom yes) (on_board yes) (dnp no) (fields_autoplaced)
-    (property "Reference" "#PWR044" (at 204.47 118.11 0)
+    (property "Reference" "#PWR046" (at 204.47 118.11 0)
       (effects (font (size 1.27 1.27)) hide)
     )
@@
       (project "tsukuba_challenge"
         (path "/55f88ae9-9831-47be-a185-734020e38c84/9c1fd94d-8d77-4c45-be6e-46f605b5b044"
-          (reference "#PWR044") (unit 1)
-        )
-      )
+          (reference "#PWR046") (unit 1)
+        )
+      )

Commit message: 4/13 product update
Parts:
- FB1, FB2, FB3, FB4, FB5: LCSC (none) -> C596498
- IC1: LCSC (none) -> C3234830
Changed lines of the file:
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@@
+      (effects (font (size 1.27 1.27)) hide)
+    )
+    (property "LCSC" "C596498" (at 105.41 57.15 0)
       (effects (font (size 1.27 1.27)) hide)
     )
@@
       (effects (font (size 1.27 1.27)) hide)
     )
+    (property "LCSC" "C596498" (at 81.28 87.63 0)
+      (effects (font (size 1.27 1.27)) hide)
+    )
     (pin "1")
     (pin "2")
@@
       (effects (font (size 1.27 1.27)) hide)
     )
+    (property "LCSC" "C596498" (at 80.01 102.87 0)
+      (effects (font (size 1.27 1.27)) hide)
+    )
     (pin "1")
     (pin "2")
@@
     )
     (property "Datasheet" "~" (at 198.12 102.87 0)
+      (effects (font (size 1.27 1.27)) hide)
+    )
+    (property "LCSC" "C596498" (at 198.12 102.87 0)
       (effects (font (size 1.27 1.27)) hide)
     )
@@
     (property "Manufacturer_Part_Number" "ISOW1044BDFMR" (at 154.94 862.23 0)
       (effects (font (size 1.27 1.27)) (justify left top) hide)
+    )
+    (property "LCSC" "C3234830" (at 123.19 67.31 0)
+      (effects (font (size 1.27 1.27)) hide)
     )
     (pin "1")
@@
       (effects (font (size 1.27 1.27)) hide)
     )
+    (property "LCSC" "C596498" (at 198.12 87.63 0)
+      (effects (font (size 1.27 1.27)) hide)
+    )

Commit message: 6/29
Parts:
- C10, C4: LCSC (none) -> C15849
- C11, C3, C9: LCSC (none) -> C19702
- C5, C8: LCSC (none) -> C57112
- C6, C7: LCSC (none) -> C14663
- R3: LCSC (none) -> C23162
Changed lines of the file:
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@@
+      (effects (font (size 1.27 1.27)) hide)
+    )
+    (property "LCSC" "C15849" (at 101.6 95.25 0)
       (effects (font (size 1.27 1.27)) hide)
     )
@@
       (effects (font (size 1.27 1.27)) hide)
     )
+    (property "LCSC" "C19702" (at 189.23 95.25 0)
+      (effects (font (size 1.27 1.27)) hide)
+    )
     (pin "1")
     (pin "2")
@@
     )
     (property "Datasheet" "~" (at 110.49 63.5 0)
+      (effects (font (size 1.27 1.27)) hide)
+    )
+    (property "LCSC" "C14663" (at 110.49 63.5 0)
       (effects (font (size 1.27 1.27)) hide)
     )
@@
       (effects (font (size 1.27 1.27)) hide)
     )
+    (property "LCSC" "C14663" (at 168.91 62.23 0)
+      (effects (font (size 1.27 1.27)) hide)
+    )
     (pin "1")
     (pin "2")
@@
       (effects (font (size 1.27 1.27)) hide)
     )
+    (property "LCSC" "C19702" (at 176.53 62.23 0)
+      (effects (font (size 1.27 1.27)) hide)
+    )
     (pin "1")
     (pin "2")
@@
       (effects (font (size 1.27 1.27)) hide)
     )
+    (property "LCSC" "C57112" (at 172.72 95.25 0)
+      (effects (font (size 1.27 1.27)) hide)
+    )
     (pin "1")
     (pin "2")
@@
       (effects (font (size 1.27 1.27)) hide)
     )
+    (property "LCSC" "C15849" (at 180.34 95.25 0)
+      (effects (font (size 1.27 1.27)) hide)
+    )
     (pin "1")
     (pin "2")
@@
       (effects (font (size 1.27 1.27)) hide)
     )
+    (property "LCSC" "C57112" (at 109.22 95.25 0)
+      (effects (font (size 1.27 1.27)) hide)
+    )
     (pin "1")
     (pin "2")
@@
     )
     (property "Datasheet" "~" (at 91.44 95.25 0)
+      (effects (font (size 1.27 1.27)) hide)
+    )
+    (property "LCSC" "C19702" (at 91.44 95.25 0)
       (effects (font (size 1.27 1.27)) hide)
     )
@@
       (effects (font (size 1.27 1.27)) hide)
     )
+    (property "LCSC" "C23162" (at 93.98 63.5 0)
+      (effects (font (size 1.27 1.27)) hide)
+    )
