File: STM32F302.kicad_sch (KiCad schematic)
At the start: 15 parts, among them SW1 SPST_SW, U2 STM32F302CBTx, Y1 12MHz

Commit message: 6/29
Parts:
- C10, C11: LCSC (none) -> C1634
- C2: LCSC (none) -> C19702
- C3, C4, C5, C6, C8, C9: LCSC (none) -> C14663
- C7: LCSC (none) -> C15849
- R9: LCSC (none) -> C25804
- U2: LCSC (none) -> C94046
Connections:
- net EMS_OBSERVE: now also U2.12 (PA2); no longer U2.41 (PB5)
- net INDICATOR_BUZZER: now also U2.25 (PB12); no longer U2.26 (PB13)
- net INDICATOR_GREEN: now also U2.26 (PB13); no longer U2.25 (PB12)
- net INDICATOR_RED: now also U2.28 (PB15); no longer U2.21 (PB10)
- net INDICATOR_YELLOW: now also U2.27 (PB14); no longer U2.22 (PB11)
Changed lines of the file:
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@@
   (no_connect (at 95.25 105.41))
   (no_connect (at 95.25 97.79))
-  (no_connect (at 95.25 140.97))
   (no_connect (at 128.27 77.47))
   (no_connect (at 95.25 95.25))
   (no_connect (at 128.27 87.63))
-  (no_connect (at 95.25 138.43))
   (no_connect (at 95.25 92.71))
   (no_connect (at 128.27 82.55))
   (no_connect (at 95.25 120.65))
   (no_connect (at 128.27 74.93))
-  (no_connect (at 128.27 80.01))
+  (no_connect (at 95.25 115.57))
+  (no_connect (at 95.25 130.81))
+  (no_connect (at 95.25 128.27))
   (no_connect (at 95.25 107.95))
   (no_connect (at 128.27 92.71))
@@
     (effects (font (size 1.27 1.27)) (justify left))
   )
-  (hierarchical_label "INDICATOR_BUZZER" (shape output) (at 95.25 135.89 180) (fields_autoplaced)
+  (hierarchical_label "INDICATOR_BUZZER" (shape output) (at 95.25 133.35 180) (fields_autoplaced)
     (effects (font (size 1.27 1.27)) (justify right))
   )
@@
     (effects (font (size 1.27 1.27)) (justify left))
   )
-  (hierarchical_label "INDICATOR_YELLOW" (shape output) (at 95.25 130.81 180) (fields_autoplaced)
+  (hierarchical_label "INDICATOR_YELLOW" (shape output) (at 95.25 138.43 180) (fields_autoplaced)
     (effects (font (size 1.27 1.27)) (justify right))
   )
@@
     (effects (font (size 1.27 1.27)) (justify right))
   )
-  (hierarchical_label "INDICATOR_RED" (shape output) (at 95.25 128.27 180) (fields_autoplaced)
+  (hierarchical_label "INDICATOR_RED" (shape output) (at 95.25 140.97 180) (fields_autoplaced)
     (effects (font (size 1.27 1.27)) (justify right))
   )
@@
     (effects (font (size 1.27 1.27)) (justify left))
   )
-  (hierarchical_label "INDICATOR_GREEN" (shape output) (at 95.25 133.35 180) (fields_autoplaced)
+  (hierarchical_label "INDICATOR_GREEN" (shape output) (at 95.25 135.89 180) (fields_autoplaced)
     (effects (font (size 1.27 1.27)) (justify right))
   )
@@
     (effects (font (size 1.27 1.27)) (justify right))
   )
-  (hierarchical_label "EMS_OBSERVE" (shape input) (at 95.25 115.57 180) (fields_autoplaced)
-    (effects (font (size 1.27 1.27)) (justify right))
+  (hierarchical_label "EMS_OBSERVE" (shape input) (at 128.27 80.01 0) (fields_autoplaced)
+    (effects (font (size 1.27 1.27)) (justify left))
   )
   (symbol (lib_id "Switch:SW_SPST") (at 29.21 86.36 90) (unit 1)
@@
       (effects (font (size 1.27 1.27)) hide)
     )
+    (property "LCSC" "C25804" (at 45.72 86.36 0)
+      (effects (font (size 1.27 1.27)) hide)
+    )
     (pin "1")
     (pin "2")
@@
       (effects (font (size 1.27 1.27)) hide)
     )
+    (property "LCSC" "C14663" (at 184.15 33.02 0)
+      (effects (font (size 1.27 1.27)) hide)
+    )
     (pin "1")
     (pin "2")
@@
       (effects (font (size 1.27 1.27)) hide)
     )
+    (property "LCSC" "C14663" (at 182.88 81.28 0)
+      (effects (font (size 1.27 1.27)) hide)
+    )
     (pin "1")
     (pin "2")
@@
       (effects (font (size 1.27 1.27)) hide)
     )
+    (property "LCSC" "C14663" (at 173.99 33.02 0)
+      (effects (font (size 1.27 1.27)) hide)
+    )
     (pin "1")
     (pin "2")
@@
       (effects (font (size 1.27 1.27)) hide)
     )
+    (property "LCSC" "C14663" (at 195.58 33.02 0)
+      (effects (font (size 1.27 1.27)) hide)
+    )
     (pin "1")
     (pin "2")
@@
       (effects (font (size 1.27 1.27)) hide)
     )
+    (property "LCSC" "C14663" (at 35.56 86.36 0)
+      (effects (font (size 1.27 1.27)) hide)
+    )
     (pin "1")
     (pin "2")
@@
       (effects (font (size 1.27 1.27)) hide)
     )
+    (property "LCSC" "C14663" (at 163.83 33.02 0)
+      (effects (font (size 1.27 1.27)) hide)
+    )
     (pin "1")
     (pin "2")
@@
     )
     (property "Datasheet" "https://www.st.com/resource/en/datasheet/stm32f302cb.pdf" (at 110.49 110.49 0)
+      (effects (font (size 1.27 1.27)) hide)
+    )
+    (property "LCSC" "C94046" (at 110.49 110.49 0)
       (effects (font (size 1.27 1.27)) hide)
     )
@@
       (effects (font (size 1.27 1.27)) hide)
     )
+    (property "LCSC" "C1634" (at 55.88 113.03 0)
+      (effects (font (size 1.27 1.27)) hide)
+    )
     (pin "1")
     (pin "2")
@@
       (effects (font (size 1.27 1.27)) hide)
     )
+    (property "LCSC" "C15849" (at 172.72 81.28 0)
+      (effects (font (size 1.27 1.27)) hide)
+    )
     (pin "1")
     (pin "2")
@@
       (effects (font (size 1.27 1.27)) hide)
     )
+    (property "LCSC" "C19702" (at 153.67 33.02 0)
+      (effects (font (size 1.27 1.27)) hide)
+    )
     (pin "1")
     (pin "2")
@@
       (effects (font (size 1.27 1.27)) hide)
     )
+    (property "LCSC" "C1634" (at 67.31 113.03 0)
+      (effects (font (size 1.27 1.27)) hide)
+    )
