File: tsukuba_challenge.kicad_sch (KiCad schematic)
At the start: 9 parts, among them J1 stlink, J6 PWR_BATT, J7 COMPUTER_BATT, J8 COMPUTER, J9 USB_C_Receptacle, U3 USBLC6-2SC6

Commit message: 3/30
Parts:
- added D7: LED, symbol Device:LED
- added J4: INDICATOR, symbol Connector_Generic:Conn_01x08
- added J5, J6: CAN, symbol Connector_Generic:Conn_01x02
- added Q1: TBD62083AFWG_Z,EHZ, my_pretty:SOIC127P1032X285-18N, symbol my_library:TBD62083AFWG_Z,EHZ
- added R18: 1.2k, symbol Device:R
- added R3, R4: 120, Resistor_SMD:R_0805_2012Metric, symbol Device:R
- J3: renamed from J1; value stlink -> ST-LINK; footprint (none) -> my_pretty:JTAG_BOX_CONN
- J7: value COMPUTER_BATT -> CAN
- J8: value COMPUTER -> CAN
- renumbered C16 to C1, J6 to J1, J9 to J2, R9 to R1, R10 to R2, U3 to U1
Connections:
- net D+_IN: now also J2.A6 (D+), J2.B6 (D+)
- net D-_IN: now also J2.A7 (D-), J2.B7 (D-)
- net GND: now also J2.A1 (GND), J2.A12 (GND), J2.B1 (GND), J2.B12 (GND), J2.S1 (SHIELD), R1.2, R2.2, D7.1 (K), Q1.9 (GND); no longer J7.1 (Pin_1), J8.1 (Pin_1)
- net MCU_CYCLE_LED: now also R18.1
- net CAN_Transceiver/CAN_L: now reaches J7.2 (Pin_2), J8.2 (Pin_2)
- net CAN_Transceiver/CAN_L: now also J5.2 (Pin_2), J6.2 (Pin_2), R3.2, R4.2
- new net: D7.2 (A), R18.2
- new net: J4.2 (Pin_2), Q1.18 (O1)
- new net: J4.3 (Pin_3), Q1.17 (O2)
- new net: J4.4 (Pin_4), Q1.16 (O3)
- new net: J4.5 (Pin_5), Q1.15 (O4)
- new net +12V: J4.8 (Pin_8), Q1.10 (COMMON)
- new net CAN_Transceiver/CAN_H: J5.1 (Pin_1), J6.1 (Pin_1), J7.1 (Pin_1), J8.1 (Pin_1), R3.1, R4.1
- new net STM32F103/INDICATOR_BUZZER: Q1.4 (I4)
- new net STM32F103/INDICATOR_GREEN: Q1.3 (I3)
- new net STM32F103/INDICATOR_RED: Q1.1 (I1)
- new net STM32F103/INDICATOR_YELLOW: Q1.2 (I2)
- no-connect marks 8 -> 30
Other:
- added sheet CAN_Transceiver (CAN_Transceiver.kicad_sch)
- sheet STM32F103 ports: added INDICATOR_BUZZER, INDICATOR_GREEN, INDICATOR_RED, INDICATOR_YELLOW; removed none
- moved on the sheet: C1, J2, J3, R1, R2, U1

Commit message: 4/2
Parts:
- removed J2: USB_C_Receptacle, Connector_USB:USB_C_Receptacle_GCT_USB4105-xx-A_16P_TopMnt_Horizontal, symbol Connector:USB_C_Receptacle
- removed J4: INDICATOR, symbol Connector_Generic:Conn_01x08
- added H1, H2, H3, H4: MountingHole, MountingHole:MountingHole_3.2mm_M3, symbol Mechanical:MountingHole
- added J2: USB_C_Receptacle_USB2.0_16P, Connector_USB:USB_C_Receptacle_G-Switch_GT-USB-7010ASV, symbol Connector:USB_C_Receptacle_USB2.0_16P
- added J4, J5, J6: INDICATOR, TerminalBlock:TerminalBlock_bornier-2_P5.08mm, symbol Connector_Generic:Conn_01x02
- added R3: 1.5k, Resistor_SMD:R_0603_1608Metric, symbol Device:R
- added R4, R5: 22, Resistor_SMD:R_0603_1608Metric, symbol Device:R
- C1: footprint (none) -> Capacitor_SMD:C_0603_1608Metric
- D1: renamed from D7; footprint (none) -> LED_SMD:LED_0603_1608Metric
- J1: footprint (none) -> Connector_AMASS:AMASS_XT60-M_1x02_P7.20mm_Vertical
- J10: renamed from J8; footprint (none) -> Connector_JST:JST_XA_B02B-XASK-1_1x02_P2.50mm_Vertical
- J7: renamed from J5; footprint (none) -> Connector_JST:JST_XA_B02B-XASK-1_1x02_P2.50mm_Vertical
- J8: renamed from J6; footprint (none) -> Connector_JST:JST_XA_B02B-XASK-1_1x02_P2.50mm_Vertical
- J9: renamed from J7; footprint (none) -> Connector_JST:JST_XA_B02B-XASK-1_1x02_P2.50mm_Vertical
- R1, R2: footprint (none) -> Resistor_SMD:R_0603_1608Metric
- R6: renamed from R18; footprint (none) -> Resistor_SMD:R_0603_1608Metric
- R7: renamed from R3; footprint Resistor_SMD:R_0805_2012Metric -> Resistor_SMD:R_0603_1608Metric
- R8: renamed from R4; footprint Resistor_SMD:R_0805_2012Metric -> Resistor_SMD:R_0603_1608Metric
Connections:
- net +12V: now also J6.2 (Pin_2)
- net +3.3V: now also R3.1
- net D+_IN: now also J2.A6 (D+), J2.B6 (D+)
- net D+_OUT: now also R4.1
- net D-_IN: now also J2.A7 (D-), J2.B7 (D-)
- net D-_OUT: now also R5.1
- net GND: now also J2.A1 (GND), J2.A12 (GND), J2.B1 (GND), J2.B12 (GND), J2.S1 (SHIELD)
- net at R1.1: now also J2.A5 (CC1)
- net at R2.1: now also J2.B5 (CC2)
- net at Q1.18 (O1): now also J4.1 (Pin_1)
- net at Q1.17 (O2): now also J4.2 (Pin_2)
- net at Q1.16 (O3): now also J5.1 (Pin_1)
- net at Q1.15 (O4): now also J5.2 (Pin_2)
- new net: J2.A4 (VBUS), J2.A9 (VBUS), J2.B4 (VBUS), J2.B9 (VBUS)
- new net STM32F103/USB_D+: R3.2, R4.2
- new net STM32F103/USB_D-: R5.2
- no-connect marks 30 -> 20
Other:
- sheet STM32F103 ports: added USB_D+, USB_D-; removed none
- moved on the sheet: C1, J3

Commit message: 4/12
Parts:
- removed J2: USB_C_Receptacle_USB2.0_16P, Connector_USB:USB_C_Receptacle_G-Switch_GT-USB-7010ASV, symbol Connector:USB_C_Receptacle_USB2.0_16P
- added J2: USB_C_Receptacle_USB2.0, Connector_USB:USB_C_Receptacle_G-Switch_GT-USB-7010ASV, symbol Connector:USB_C_Receptacle_USB2.0
- D1: value LED -> LED_MCU
Connections:
- net D+_IN: now also J2.A6 (D+), J2.B6 (D+)
- net D-_IN: now also J2.A7 (D-), J2.B7 (D-)
- net GND: now also J2.A1 (GND), J2.A12 (GND), J2.B1 (GND), J2.B12 (GND), J2.S1 (SHIELD)
- net at R1.1: now also J2.A5 (CC1)
- net at R2.1: now also J2.B5 (CC2)
- new net: J2.A4 (VBUS), J2.A9 (VBUS), J2.B4 (VBUS), J2.B9 (VBUS)
Other:
- moved on the sheet: C1

Commit message: 4/13 product update
Parts:
- D1: LCSC (none) -> C2290
- H1, H2, H3, H4, J1, J10, J3, J4, J5, J6, J7, J8, J9: now left out of the parts list
- J2: JLCPCB Position Offset (none) -> 0,1.3; LCSC (none) -> C2988369
- Q1: JLCPCB Rotation Offset (none) -> -90; LCSC (none) -> C108880
- U1: JLCPCB Rotation Offset (none) -> 90; LCSC (none) -> C7519

Commit message: ✨feat:f302
Parts:
- H1, H2, H3, H4: footprint MountingHole:MountingHole_3.2mm_M3 -> MountingHole:MountingHole_4.3mm_M4
- R4: value 22 -> 33k
- R5: value 22 -> 82k
Connections:
- net +3.3V: no longer R3.1
- net D+_OUT: now also R3.1; no longer R4.1
- net D-_OUT: no longer R5.1
- net GND: now also R5.1
- net USB_VBUS: now reaches J2.A4 (VBUS), J2.A9 (VBUS), J2.B4 (VBUS), J2.B9 (VBUS)
- net USB_VBUS: now also R4.1
- net STM32F302/USB_D+ renamed STM32F302/USB_PULLUP
- net STM32F302/USB_PULLUP: no longer R4.2
- net STM32F302/USB_D- renamed STM32F302/USB_VBUS
- net STM32F302/USB_VBUS: now also R4.2
- no-connect marks 20 -> 19
Other:
- sheet STM32F103 renamed STM32F302
- sheet STM32F302: file STM32F103.kicad_sch -> STM32F302.kicad_sch
- sheet STM32F302 ports: added USB_PULLUP, USB_VBUS; removed none
- moved on the sheet: R3, R4, R5

Commit message: 6/29
Parts:
- C1: LCSC (none) -> C14663
- R1, R2: LCSC (none) -> C23186
- R3: LCSC (none) -> C22843
- R4: LCSC (none) -> C4216
- R5: LCSC (none) -> C23254
- R6: LCSC (none) -> C22765
- R7, R8: LCSC (none) -> C22787
Connections:
- net D+_IN: now also U1.3 (I/O2); no longer U1.1 (I/O1)
- net D+_OUT: now also U1.4 (I/O2); no longer U1.6 (I/O1)
- net D-_IN: now also U1.1 (I/O1); no longer U1.3 (I/O2)
- net D-_OUT: now also U1.6 (I/O1); no longer U1.4 (I/O2)
