File: tsukuba_challenge.kicad_sch (KiCad schematic)
At the start: 26 parts, among them J1 PWR_BATT, J10 CAN, J2 USB_C_Receptacle_USB2.0, J3 ST-LINK, J4 INDICATOR, J5 INDICATOR, J6 INDICATOR, J7 CAN, J8 CAN, J9 CAN, Q1 TBD62083AFWG_Z,EHZ, U1 USBLC6-2SC6

Commit message: 7/19
Connections:
- net GND: now also J6.1 (Pin_1)
- no-connect marks 19 -> 18
